Commit message: done

File: body0.urdf (robot description, URDF)
Before this commit: robot robot, 12 links, 11 joints
Links:
- removed link Link10
- removed link Link11
- link Link8: geometry collision box size=0.25891675029296335 0.5112747213686085 0.4049341374504143; visual box size=0.25891675029296335 0.5112747213686085 0.4049341374504143
- link Link9: geometry collision box size=0.47214271545271336 0.1007012080683658 0.4341718354537837; visual box size=0.47214271545271336 0.1007012080683658 0.4341718354537837
Joints:
- removed joint Link0_Link2
- removed joint Link1_Link6
- removed joint Link1_Link9
- removed joint Link2_Link5
- removed joint Link3_Link10
- removed joint Link3_Link4
- removed joint Link5_Link7
- removed joint Link5_Link8
- removed joint Link9_Link11
- added joint Link0_Link5: type revolute, parent Link0, child Link5, origin xyz=0.3054434867219008 0.2768062065673212 7.449707056431781 rpy=0 0 0, axis 0 1 0, limit lower=-3.14159 upper=3.14159 effort=0.0 velocity=0.0
- added joint Link0_Link7: type revolute, parent Link0, child Link7, origin xyz=0.30130262209425407 0.34245883926692045 7.983303183885379 rpy=0 0 0, axis 0 1 0, limit lower=-3.14159 upper=3.14159 effort=0.0 velocity=0.0
- added joint Link1_Link2: type revolute, parent Link1, child Link2, origin xyz=0.03447003119734737 0.44941914398399674 -0.6213090513207824 rpy=0 0 0, axis 0 0 1, limit lower=-3.14159 upper=3.14159 effort=0.0 velocity=0.0
- added joint Link1_Link8: type revolute, parent Link1, child Link8, origin xyz=-0.3649158741300643 0.37953422528590697 -0.5449971298908969 rpy=0 0 0, axis 0 0 1, limit lower=-3.14159 upper=3.14159 effort=0.0 velocity=0.0
- added joint Link2_Link4: type revolute, parent Link2, child Link4, origin xyz=0.42221092576252406 0.22005652464963757 -0.13063317996966298 rpy=0 0 0, axis 1 0 0, limit lower=-3.14159 upper=3.14159 effort=0.0 velocity=0.0
- added joint Link4_Link6: type revolute, parent Link4, child Link6, origin xyz=0.7103744664517335 0.45108297521979135 0.10621320579548385 rpy=0 0 0, axis 0 1 0, limit lower=-3.14159 upper=3.14159 effort=0.0 velocity=0.0
- added joint Link6_Link9: type revolute, parent Link6, child Link9, origin xyz=0.05171678941556378 0.6332620642774094 -0.3091844983376658 rpy=0 0 0, axis 0 0 1, limit lower=-3.14159 upper=3.14159 effort=0.0 velocity=0.0
- joint Link0_Link1: axis 0 1 0 -> 1 0 0; origin xyz=-0.3054434867219008 0.04331407641852992 9.303965672510301 rpy=0 0 0 -> xyz=-0.23882146929074846 0.04680756234974069 7.016696816114621 rpy=0 0 0
- joint Link2_Link3: axis 0 0 1 -> 0 1 0; origin xyz=0.42221092576252406 0.05236346826659599 0.07516621809888827 rpy=0 0 0 -> xyz=-0.3943682981346013 0.7579544029403025 -0.10091353964101608 rpy=0 0 0

File: body1.urdf (robot description, URDF)
Before this commit: robot robot, 12 links, 11 joints
Links:
- removed link Link10
- removed link Link11
- link Link8: geometry collision box size=0.25891675029296335 0.5112747213686085 0.4049341374504143; visual box size=0.25891675029296335 0.5112747213686085 0.4049341374504143
- link Link9: geometry collision box size=0.47214271545271336 0.1007012080683658 0.4341718354537837; visual box size=0.47214271545271336 0.1007012080683658 0.4341718354537837
Joints:
- removed joint Link0_Link2
- removed joint Link1_Link6
- removed joint Link1_Link9
- removed joint Link2_Link5
- removed joint Link3_Link10
- removed joint Link3_Link4
- removed joint Link5_Link7
- removed joint Link5_Link8
- removed joint Link9_Link11
- added joint Link0_Link5: type revolute, parent Link0, child Link5, origin xyz=0.3054434867219008 0.2768062065673212 7.449707056431781 rpy=0 0 0, axis 0 1 0, limit lower=-3.14159 upper=3.14159 effort=0.0 velocity=0.0
- added joint Link0_Link7: type revolute, parent Link0, child Link7, origin xyz=0.30130262209425407 0.34245883926692045 7.983303183885379 rpy=0 0 0, axis 0 1 0, limit lower=-3.14159 upper=3.14159 effort=0.0 velocity=0.0
- added joint Link1_Link2: type revolute, parent Link1, child Link2, origin xyz=0.03447003119734737 0.44941914398399674 -0.6213090513207824 rpy=0 0 0, axis 0 0 1, limit lower=-3.14159 upper=3.14159 effort=0.0 velocity=0.0
- added joint Link1_Link8: type revolute, parent Link1, child Link8, origin xyz=-0.3649158741300643 0.37953422528590697 -0.5449971298908969 rpy=0 0 0, axis 0 0 1, limit lower=-3.14159 upper=3.14159 effort=0.0 velocity=0.0
- added joint Link2_Link4: type revolute, parent Link2, child Link4, origin xyz=0.42221092576252406 0.22005652464963757 -0.13063317996966298 rpy=0 0 0, axis 1 0 0, limit lower=-3.14159 upper=3.14159 effort=0.0 velocity=0.0
- added joint Link4_Link6: type revolute, parent Link4, child Link6, origin xyz=0.7103744664517335 0.45108297521979135 0.10621320579548385 rpy=0 0 0, axis 0 1 0, limit lower=-3.14159 upper=3.14159 effort=0.0 velocity=0.0
- added joint Link6_Link9: type revolute, parent Link6, child Link9, origin xyz=0.05171678941556378 0.6332620642774094 -0.3091844983376658 rpy=0 0 0, axis 0 0 1, limit lower=-3.14159 upper=3.14159 effort=0.0 velocity=0.0
- joint Link0_Link1: axis 0 1 0 -> 1 0 0; origin xyz=-0.3054434867219008 0.04331407641852992 9.303965672510301 rpy=0 0 0 -> xyz=-0.23882146929074846 0.04680756234974069 7.016696816114621 rpy=0 0 0
- joint Link2_Link3: axis 0 0 1 -> 0 1 0; origin xyz=0.42221092576252406 0.05236346826659599 0.07516621809888827 rpy=0 0 0 -> xyz=-0.3943682981346013 0.7579544029403025 -0.10091353964101608 rpy=0 0 0

Commit message: new commit

File: body0.urdf (robot description, URDF)
Before this commit: robot robot, 10 links, 9 joints
Links:
- removed link Link8
- removed link Link9
- link Link0: geometry collision box size=0.7298317482601286 0.8988382879679935 0.6839839319154413; visual box size=0.7298317482601286 0.8988382879679935 0.6839839319154413
- link Link1: geometry collision box size=0.8444218515250481 0.7579544029403025 0.420571580830845; visual box size=0.8444218515250481 0.7579544029403025 0.420571580830845
- link Link2: geometry collision box size=0.5833820394550312 0.9081128851953352 0.5046868558173903; visual box size=0.5833820394550312 0.9081128851953352 0.5046868558173903
- link Link3: geometry collision box size=0.8102172359965896 0.9021659504395827 0.3101475693193326; visual box size=0.8102172359965896 0.9021659504395827 0.3101475693193326
- link Link4: geometry collision box size=0.25050634136244054 0.9097462559682401 0.9827854760376531; visual box size=0.25050634136244054 0.9097462559682401 0.9827854760376531
- link Link5: geometry collision box size=0.28183784439970383 0.7558042041572239 0.6183689966753316; visual box size=0.28183784439970383 0.7558042041572239 0.6183689966753316
- link Link6: geometry collision box size=0.7837985890347726 0.30331272607892745 0.4765969541523558; visual box size=0.7837985890347726 0.30331272607892745 0.4765969541523558
- link Link7: geometry collision box size=0.25891675029296335 0.5112747213686085 0.4049341374504143; visual box size=0.25891675029296335 0.5112747213686085 0.4049341374504143
Joints:
- removed joint Link0_Link5
- removed joint Link0_Link7
- removed joint Link1_Link2
- removed joint Link1_Link8
- removed joint Link2_Link3
- removed joint Link2_Link4
- removed joint Link6_Link9
- added joint Link0_Link2: type revolute, parent Link0, child Link2, origin xyz=0.15344962375102444 0.25621184024907806 5.658008034042279 rpy=0 0 0, axis 1 0 0, limit lower=-3.14159 upper=3.14159 effort=0.0 velocity=0.0
- added joint Link1_Link3: type revolute, parent Link1, child Link3, origin xyz=-0.4276339156526157 0.2786261422178288 0.2102857904154225 rpy=0 0 0, axis 0 0 1, limit lower=-3.14159 upper=3.14159 effort=0.0 velocity=0.0
- added joint Link2_Link5: type revolute, parent Link2, child Link5, origin xyz=-0.18022591021410994 -0.45405644259766764 -0.38426053305662794 rpy=0 0 0, axis 0 1 0, limit lower=-3.14159 upper=3.14159 effort=0.0 velocity=0.0
- added joint Link3_Link4: type revolute, parent Link3, child Link4, origin xyz=-0.042155950019190175 -0.378507496866453 0.3101475693193326 rpy=0 0 0, axis 0 0 1, limit lower=-3.14159 upper=3.14159 effort=0.0 velocity=0.0
- added joint Link5_Link7: type revolute, parent Link5, child Link7, origin xyz=0.14091892219985191 -0.15159383239048466 0.029205633569223483 rpy=0 0 0, axis 0 0 1, limit lower=-3.14159 upper=3.14159 effort=0.0 velocity=0.0
- joint Link0_Link1: axis 1 0 0 -> 0 0 1; origin xyz=-0.23882146929074846 0.04680756234974069 7.016696816114621 rpy=0 0 0 -> xyz=-0.3649158741300643 0.3739117665281173 5.7218044905591245 rpy=0 0 0
- joint Link4_Link6: axis 0 1 0 -> 1 0 0; origin xyz=0.7103744664517335 0.45108297521979135 0.10621320579548385 rpy=0 0 0 -> xyz=-0.09793348870015077 0.45487312798412005 0.6943982915458664 rpy=0 0 0

File: body1.urdf (robot description, URDF)
Before this commit: robot robot, 10 links, 9 joints
Links:
- removed link Link8
- removed link Link9
- link Link0: geometry collision box size=0.7298317482601286 0.8988382879679935 0.6839839319154413; visual box size=0.7298317482601286 0.8988382879679935 0.6839839319154413
- link Link1: geometry collision box size=0.8444218515250481 0.7579544029403025 0.420571580830845; visual box size=0.8444218515250481 0.7579544029403025 0.420571580830845
- link Link2: geometry collision box size=0.5833820394550312 0.9081128851953352 0.5046868558173903; visual box size=0.5833820394550312 0.9081128851953352 0.5046868558173903
- link Link3: geometry collision box size=0.8102172359965896 0.9021659504395827 0.3101475693193326; visual box size=0.8102172359965896 0.9021659504395827 0.3101475693193326
- link Link4: geometry collision box size=0.25050634136244054 0.9097462559682401 0.9827854760376531; visual box size=0.25050634136244054 0.9097462559682401 0.9827854760376531
- link Link5: geometry collision box size=0.28183784439970383 0.7558042041572239 0.6183689966753316; visual box size=0.28183784439970383 0.7558042041572239 0.6183689966753316
- link Link6: geometry collision box size=0.7837985890347726 0.30331272607892745 0.4765969541523558; visual box size=0.7837985890347726 0.30331272607892745 0.4765969541523558
- link Link7: geometry collision box size=0.25891675029296335 0.5112747213686085 0.4049341374504143; visual box size=0.25891675029296335 0.5112747213686085 0.4049341374504143
Joints:
- removed joint Link0_Link5
- removed joint Link0_Link7
- removed joint Link1_Link2
- removed joint Link1_Link8
- removed joint Link2_Link3
- removed joint Link2_Link4
- removed joint Link6_Link9
- added joint Link0_Link2: type revolute, parent Link0, child Link2, origin xyz=0.15344962375102444 0.25621184024907806 5.658008034042279 rpy=0 0 0, axis 1 0 0, limit lower=-3.14159 upper=3.14159 effort=0.0 velocity=0.0
- added joint Link1_Link3: type revolute, parent Link1, child Link3, origin xyz=-0.4276339156526157 0.2786261422178288 0.2102857904154225 rpy=0 0 0, axis 0 0 1, limit lower=-3.14159 upper=3.14159 effort=0.0 velocity=0.0
- added joint Link2_Link5: type revolute, parent Link2, child Link5, origin xyz=-0.18022591021410994 -0.45405644259766764 -0.38426053305662794 rpy=0 0 0, axis 0 1 0, limit lower=-3.14159 upper=3.14159 effort=0.0 velocity=0.0
- added joint Link3_Link4: type revolute, parent Link3, child Link4, origin xyz=-0.042155950019190175 -0.378507496866453 0.3101475693193326 rpy=0 0 0, axis 0 0 1, limit lower=-3.14159 upper=3.14159 effort=0.0 velocity=0.0
- added joint Link5_Link7: type revolute, parent Link5, child Link7, origin xyz=0.14091892219985191 -0.15159383239048466 0.029205633569223483 rpy=0 0 0, axis 0 0 1, limit lower=-3.14159 upper=3.14159 effort=0.0 velocity=0.0
- joint Link0_Link1: axis 1 0 0 -> 0 0 1; origin xyz=-0.23882146929074846 0.04680756234974069 7.016696816114621 rpy=0 0 0 -> xyz=-0.3649158741300643 0.3739117665281173 5.7218044905591245 rpy=0 0 0
- joint Link4_Link6: axis 0 1 0 -> 1 0 0; origin xyz=0.7103744664517335 0.45108297521979135 0.10621320579548385 rpy=0 0 0 -> xyz=-0.09793348870015077 0.45487312798412005 0.6943982915458664 rpy=0 0 0

Commit message: finished

File: body0.urdf (robot description, URDF)
Before this commit: robot robot, 8 links, 7 joints
Links:
- removed link Link4
- removed link Link5
- removed link Link6
- removed link Link7
- link Link0: geometry collision box size=0.8444218515250481 0.7579544029403025 0.420571580830845; visual box size=0.8444218515250481 0.7579544029403025 0.420571580830845
- link Link1: geometry collision box size=0.5833820394550312 0.9081128851953352 0.5046868558173903; visual box size=0.5833820394550312 0.9081128851953352 0.5046868558173903
- link Link2: geometry collision box size=0.7837985890347726 0.30331272607892745 0.4765969541523558; visual box size=0.7837985890347726 0.30331272607892745 0.4765969541523558
- link Link3: geometry collision box size=0.25891675029296335 0.5112747213686085 0.4049341374504143; visual box size=0.25891675029296335 0.5112747213686085 0.4049341374504143
Joints:
- removed joint Link1_Link3
- removed joint Link2_Link5
- removed joint Link3_Link4
- removed joint Link4_Link6
- removed joint Link5_Link7
- added joint Link0_Link3: type revolute, parent Link0, child Link3, origin xyz=-0.42221092576252406 -0.323083799217726 3.14739933114969 rpy=0 0 0, axis 0 0 1, limit lower=-3.14159 upper=3.14159 effort=0.0 velocity=0.0
- joint Link0_Link1: axis 0 0 1 -> 1 0 0; origin xyz=-0.3649158741300643 0.3739117665281173 5.7218044905591245 rpy=0 0 0 -> xyz=-0.15520752330639082 0.10643453547468133 3.2102857904154227 rpy=0 0 0
- joint Link0_Link2: origin xyz=0.15344962375102444 0.25621184024907806 5.658008034042279 rpy=0 0 0 -> xyz=-0.023523299795879898 0.37897720147015124 2.832066275853466 rpy=0 0 0

File: body1.urdf (robot description, URDF)
Before this commit: robot robot, 8 links, 7 joints
Links:
- removed link Link4
- removed link Link5
- removed link Link6
- removed link Link7
- link Link0: geometry collision box size=0.8444218515250481 0.7579544029403025 0.420571580830845; visual box size=0.8444218515250481 0.7579544029403025 0.420571580830845
- link Link1: geometry collision box size=0.5833820394550312 0.9081128851953352 0.5046868558173903; visual box size=0.5833820394550312 0.9081128851953352 0.5046868558173903
- link Link2: geometry collision box size=0.7837985890347726 0.30331272607892745 0.4765969541523558; visual box size=0.7837985890347726 0.30331272607892745 0.4765969541523558
- link Link3: geometry collision box size=0.25891675029296335 0.5112747213686085 0.4049341374504143; visual box size=0.25891675029296335 0.5112747213686085 0.4049341374504143
Joints:
- removed joint Link1_Link3
- removed joint Link2_Link5
- removed joint Link3_Link4
- removed joint Link4_Link6
- removed joint Link5_Link7
- added joint Link0_Link3: type revolute, parent Link0, child Link3, origin xyz=-0.42221092576252406 -0.323083799217726 3.14739933114969 rpy=0 0 0, axis 0 0 1, limit lower=-3.14159 upper=3.14159 effort=0.0 velocity=0.0
- joint Link0_Link1: axis 0 0 1 -> 1 0 0; origin xyz=-0.3649158741300643 0.3739117665281173 5.7218044905591245 rpy=0 0 0 -> xyz=-0.15520752330639082 0.10643453547468133 3.2102857904154227 rpy=0 0 0
- joint Link0_Link2: origin xyz=0.15344962375102444 0.25621184024907806 5.658008034042279 rpy=0 0 0 -> xyz=-0.023523299795879898 0.37897720147015124 2.832066275853466 rpy=0 0 0
